Commit message: test commit

File: src/q4d_description/urdf/q4d.urdf.xacro (robot description, xacro)
@@ -1,4 +1,4 @@
 <robot name="q4d" xmlns:xacro="http://www.ros.org/wiki/xacro">
-	<xacro:include filename="$(find q2d_description)/urdf/q2d.urdf"/>
+<xacro:include filename="$(find q2d_description)/urdf/q2d.urdf"/>
 	<xacro:include filename="$(find q4d_description)/urdf/q4d_aux.urdf.xacro"/>
 	<xacro:include filename="$(find q4d_description)/urdf/q4d_prismatic.urdf.xacro"/>
@@ -7,11 +7,11 @@
 	<xacro:include filename="$(find q4d_description)/urdf/q4d_claw_mimic.urdf.xacro"/>
 	<xacro:aux name="aux_vertical" length="0.05" width="0.05" height="0.3" mass="0.1" parent="elbow_passive_link">
-		<origin xyz="${0.267+0.025} 0.0 0.0" rpy="0.0 0.0 0.0"/>
+		<origin xyz="${0.267+0.025} 0.0 0.1" rpy="0.0 0.0 0.0"/>
 	</xacro:aux>
-	<xacro:aux name="aux_horizontal" length="0.15" width="0.05" height="0.03" mass="0.1" parent="aux_vertical_link">
-		<origin xyz="${0.025+0.075} 0.0 ${0.15-0.015}" rpy="0.0 0.0 0.0"/>
+	<xacro:aux name="aux_horizontal" length="0.1" width="0.05" height="0.03" mass="0.1" parent="aux_vertical_link">
+		<origin xyz="${0.025+0.05} 0.0 ${0.15-0.015}" rpy="0.0 0.0 0.0"/>
 	</xacro:aux>
 	<xacro:prismatic name="prismatic" length="0.05" width="0.05" height="0.33" mass="0.1" parent="aux_horizontal_link">
-		<origin xyz="${0.075+0.025} 0.0 0.0" rpy="0.0 0.0 0.0"/>
+		<origin xyz="${0.05+0.025} 0.0 0.0" rpy="0.0 0.0 0.0"/>
 	</xacro:prismatic>
 	<xacro:revolute name="revolute" length="0.12" width="0.12" height="0.01" mass="0.1" parent="prismatic_link">
