Commit message: added cCB and hCB functions

File: install/q4d_description/share/q4d_description/urdf/q4d.urdf.xacro (robot description, xacro)
@@ -1 +1 @@
-/home/ros2/colcon_ws/src/q4d_description/urdf/q4d.urdf.xacro
+/home/ros/colcon_ws/src/q4d_description/urdf/q4d.urdf.xacro

File: install/q4d_description/share/q4d_description/urdf/q4d_aux.urdf.xacro (robot description, xacro)
@@ -1 +1 @@
-/home/ros2/colcon_ws/src/q4d_description/urdf/q4d_aux.urdf.xacro
+/home/ros/colcon_ws/src/q4d_description/urdf/q4d_aux.urdf.xacro

File: install/q4d_description/share/q4d_description/urdf/q4d_claw.urdf.xacro (robot description, xacro)
@@ -1 +1 @@
-/home/ros2/colcon_ws/src/q4d_description/urdf/q4d_claw.urdf.xacro
+/home/ros/colcon_ws/src/q4d_description/urdf/q4d_claw.urdf.xacro

File: install/q4d_description/share/q4d_description/urdf/q4d_claw_mimic.urdf.xacro (robot description, xacro)
@@ -1 +1 @@
-/home/ros2/colcon_ws/src/q4d_description/urdf/q4d_claw_mimic.urdf.xacro
+/home/ros/colcon_ws/src/q4d_description/urdf/q4d_claw_mimic.urdf.xacro

File: install/q4d_description/share/q4d_description/urdf/q4d_prismatic.urdf.xacro (robot description, xacro)
@@ -1 +1 @@
-/home/ros2/colcon_ws/src/q4d_description/urdf/q4d_prismatic.urdf.xacro
+/home/ros/colcon_ws/src/q4d_description/urdf/q4d_prismatic.urdf.xacro

File: install/q4d_description/share/q4d_description/urdf/q4d_revolute.urdf.xacro (robot description, xacro)
@@ -1 +1 @@
-/home/ros2/colcon_ws/src/q4d_description/urdf/q4d_revolute.urdf.xacro
+/home/ros/colcon_ws/src/q4d_description/urdf/q4d_revolute.urdf.xacro

File: src/install/q4d_description/share/q4d_description/urdf/q4d.urdf.xacro (robot description, xacro)
@@ -1,26 +1 @@
-<robot name="q4d" xmlns:xacro="http://www.ros.org/wiki/xacro">
-<xacro:include filename="$(find q2d_description)/urdf/q2d.urdf"/>
-	<xacro:include filename="$(find q4d_description)/urdf/q4d_aux.urdf.xacro"/>
-	<xacro:include filename="$(find q4d_description)/urdf/q4d_prismatic.urdf.xacro"/>
-	<xacro:include filename="$(find q4d_description)/urdf/q4d_revolute.urdf.xacro"/>
-	<xacro:include filename="$(find q4d_description)/urdf/q4d_claw.urdf.xacro"/>
-	<xacro:include filename="$(find q4d_description)/urdf/q4d_claw_mimic.urdf.xacro"/>
-	<xacro:aux name="aux_vertical" length="0.05" width="0.05" height="0.3" mass="0.1" parent="elbow_passive_link">
-		<origin xyz="${0.267+0.025} 0.0 0.1" rpy="0.0 0.0 0.0"/>
-	</xacro:aux>
-	<xacro:aux name="aux_horizontal" length="0.1" width="0.05" height="0.03" mass="0.1" parent="aux_vertical_link">
-		<origin xyz="${0.025+0.05} 0.0 ${0.15-0.015}" rpy="0.0 0.0 0.0"/>
-	</xacro:aux>
-	<xacro:prismatic name="prismatic" length="0.05" width="0.05" height="0.33" mass="0.1" parent="aux_horizontal_link">
-		<origin xyz="${0.05+0.025} 0.0 0.0" rpy="0.0 0.0 0.0"/>
-	</xacro:prismatic>
-	<xacro:revolute name="revolute" length="0.12" width="0.12" height="0.01" mass="0.1" parent="prismatic_link">
-		<origin xyz="0.0 0.0 ${-0.165-0.005}" rpy="0.0 0.0 0.0"/>
-	</xacro:revolute>
-	<xacro:claw name="claw" length="0.01" width="0.01" height="0.04" mass="0.1" parent="revolute_link">
-		<origin xyz="0.0 0.005 ${-0.005-0.02}" rpy="0.0 0.0 0.0"/>
-	</xacro:claw>
-	<xacro:claw_mimic name="claw_aux" length="0.01" width="0.01" height="0.04" mass="0.1" parent="revolute_link">
-		<origin xyz="0.0 -0.005 ${-0.005-0.02}" rpy="0.0 0.0 0.0"/>
-	</xacro:claw_mimic>
-</robot>
+/home/ros/colcon_ws/src/q4d_description/urdf/q4d.urdf.xacro

File: src/install/q4d_description/share/q4d_description/urdf/q4d_aux.urdf.xacro (robot description, xacro)
@@ -1,39 +1 @@
-<robot xmlns:xacro="http://www.ros.org/wiki/xacro">
-<xacro:macro name="aux" params="name length width height mass parent *origin">
-<link name="${name}_link">
-	<visual>
-		<geometry>
-			<box size="${length} ${width} ${height}"/>
-		</geometry>
-			<material name="">
-				<color rgba="0 0.0 0.0 1"/>
-			</material>
-	</visual>
-	<collision>
-		<geometry>
-			<box size="${length} ${width} ${height}"/>
-		</geometry>
-	</collision>
-	<inertial>
-		<origin xyz="0.0 0.0 0.0" rpy="0 0 0" />
-		<mass value="${mass}" />
-		<inertia
-			ixx="${mass/12*(length*length+height*height)}"
-			ixy="0.0"
-			ixz="0.0"
-			iyy="${mass/12*(width*width+height*height)}"
-			iyz="0.0"
-			izz="${mass/12*(width*width+length*length)}"/>
-		</inertial>
-</link>
-<joint name="${name}_joint" type="fixed">
-	<xacro:insert_block name="origin"/>
-	<parent link="${parent}" />
-	<child link="${name}_link" />
-	<axis xyz="0 0 1" />
-</joint>
-<gazebo reference="${name}_link">
-	<material>Gazebo/Red</material>
-</gazebo>
-</xacro:macro>
-</robot>
+/home/ros/colcon_ws/src/q4d_description/urdf/q4d_aux.urdf.xacro

File: src/install/q4d_description/share/q4d_description/urdf/q4d_claw.urdf.xacro (robot description, xacro)
@@ -1,40 +1 @@
-<robot xmlns:xacro="http://www.ros.org/wiki/xacro">
-<xacro:macro name="claw" params="name length width height mass parent *origin">
-<link name="${name}_link">
-	<visual>
-		<geometry>
-			<box size="${length} ${width} ${height}"/>
-		</geometry>
-			<material name="">
-				<color rgba="1 1 1.0 1"/>
-			</material>
-	</visual>
-	<collision>
-		<geometry>
-			<box size="${length} ${width} ${height}"/>
-		</geometry>
-	</collision>
-	<inertial>
-		<origin xyz="0.0 0.0 0.0" rpy="0 0 0" />
-		<mass value="${mass}" />
-		<inertia
-			ixx="${mass/12*(length*length+height*height)}"
-			ixy="0.0"
-			ixz="0.0"
-			iyy="${mass/12*(width*width+height*height)}"
-			iyz="0.0"
-			izz="${mass/12*(width*width+length*length)}"/>
-		</inertial>
-</link>
-<joint name="${name}_joint" type="prismatic">
-	<xacro:insert_block name="origin"/>
-	<parent link="${parent}" />
-	<child link="${name}_link" />
-	<axis xyz="0 1 0" />
-	<limit lower="0.0" upper="0.05" effort="1.0" velocity="10.0"/>
-</joint>
-<gazebo reference="${name}_link">
-	<material>Gazebo/Red</material>
-</gazebo>
-</xacro:macro>
-</robot>
+/home/ros/colcon_ws/src/q4d_description/urdf/q4d_claw.urdf.xacro

File: src/install/q4d_description/share/q4d_description/urdf/q4d_claw_mimic.urdf.xacro (robot description, xacro)
@@ -1,41 +1 @@
-<robot xmlns:xacro="http://www.ros.org/wiki/xacro">
-<xacro:macro name="claw_mimic" params="name length width height mass parent *origin">
-<link name="${name}_link">
-	<visual>
-		<geometry>
-			<box size="${length} ${width} ${height}"/>
-		</geometry>
-			<material name="">
-				<color rgba="1 1.0 1.0 1"/>
-			</material>
-	</visual>
-	<collision>
-		<geometry>
-			<box size="${length} ${width} ${height}"/>
-		</geometry>
-	</collision>
-	<inertial>
-		<origin xyz="0.0 0.0 0.0" rpy="0 0 0" />
-		<mass value="${mass}" />
-		<inertia
-			ixx="${mass/12*(length*length+height*height)}"
-			ixy="0.0"
-			ixz="0.0"
-			iyy="${mass/12*(width*width+height*height)}"
-			iyz="0.0"
-			izz="${mass/12*(width*width+length*length)}"/>
-		</inertial>
-</link>
-<joint name="${name}_joint" type="prismatic">
-	<xacro:insert_block name="origin"/>
-	<parent link="${parent}" />
-	<child link="${name}_link" />
-	<axis xyz="0 1 0" />
-	<mimic joint ="claw_joint" multiplier="-1"/>
-	<limit lower="0.0" upper="0.05" effort="1.0" velocity="10.0"/>
-</joint>
-<gazebo reference="${name}_link">
-	<material>Gazebo/Red</material>
-</gazebo>
-</xacro:macro>
-</robot>
+/home/ros/colcon_ws/src/q4d_description/urdf/q4d_claw_mimic.urdf.xacro

File: src/install/q4d_description/share/q4d_description/urdf/q4d_prismatic.urdf.xacro (robot description, xacro)
@@ -1,40 +1 @@
-<robot xmlns:xacro="http://www.ros.org/wiki/xacro">
-<xacro:macro name="prismatic" params="name length width height mass parent *origin">
-<link name="${name}_link">
-	<visual>
-		<geometry>
-			<box size="${length} ${width} ${height}"/>
-		</geometry>
-			<material name="">
-				<color rgba="0 0 0 1"/>
-			</material>
-	</visual>
-	<collision>
-		<geometry>
-			<box size="${length} ${width} ${height}"/>
-		</geometry>
-	</collision>
-	<inertial>
-		<origin xyz="0.0 0.0 0.0" rpy="0 0 0" />
-		<mass value="${mass}" />
-		<inertia
-			ixx="${mass/12*(length*length+height*height)}"
-			ixy="0.0"
-			ixz="0.0"
-			iyy="${mass/12*(width*width+height*height)}"
-			iyz="0.0"
-			izz="${mass/12*(width*width+length*length)}"/>
-		</inertial>
-</link>
-<joint name="${name}_joint" type="prismatic">
-	<xacro:insert_block name="origin"/>
-	<parent link="${parent}" />
-	<child link="${name}_link" />
-	<axis xyz="0 0 1" />
-	<limit lower="-0.15" upper="0.15" effort="1.0" velocity="10.0"/>
-</joint>
-<gazebo reference="${name}_link">
-	<material>Gazebo/Red</material>
-</gazebo>
-</xacro:macro>
-</robot>
+/home/ros/colcon_ws/src/q4d_description/urdf/q4d_prismatic.urdf.xacro

File: src/install/q4d_description/share/q4d_description/urdf/q4d_revolute.urdf.xacro (robot description, xacro)
@@ -1,38 +1 @@
-<robot xmlns:xacro="http://www.ros.org/wiki/xacro">
-<xacro:macro name="revolute" params="name length width height mass parent *origin">
-<link name="${name}_link">
-	<visual>
-		<geometry>
-			<box size="${length} ${width} ${height}"/>
-		</geometry>
-			<material name="">
-				<color rgba="0.0 1 1 1"/>
-			</material>
-	</visual>
-	<collision>
-		<geometry>
-			<box size="${length} ${width} ${height}"/>
-		</geometry>
-	</collision>
-	<inertial>
-		<origin xyz="0.0 0.0 0.0" rpy="0 0 0" />
-		<mass value="${mass}" />
-		<inertia ixx="${mass/12*(length*length+height*height)}"
-			ixy="0.0" ixz="0.0"
-			iyy="${mass/12*(width*width+height*height)}"
-			iyz="0.0"
-			izz="${mass/12*(width*width+length*length)}"/>
-	</inertial>
-</link>
-<joint name="${name}_joint" type="revolute">
-	<xacro:insert_block name="origin"/>
-	<parent link="${parent}" />
-	<child link="${name}_link" />
-	<axis xyz="0 0 1" />
-	<limit lower="-2.61799" upper="2.61799" effort="1.0" velocity="10.0"/>
-</joint>
-<gazebo reference="${name}_link">
-	<material>Gazebo/Red</material>
-</gazebo>
-</xacro:macro>
-</robot>
+/home/ros/colcon_ws/src/q4d_description/urdf/q4d_revolute.urdf.xacro
